Commit message: Changes to Motoman ES200RN 120 support package

File: motoman_es200rn_120_support/urdf/es200rn_120_macro.xacro (robot description, xacro)
@@ -1,221 +1,221 @@
 <?xml version="1.0"?>
 <robot xmlns:xacro="http://ros.org/wiki/xacro">
-<xacro:macro name="motoman_es200rn_120" params="prefix">
+  <xacro:macro name="motoman_es200rn_120" params="prefix">
     <!-- link list -->
     <link name="${prefix}base_link">
-        <visual>
-            <origin xyz="0 0 0" rpy="0 0 0"/>
-            <geometry>
-                <mesh filename="package://motoman_es200rn_120_support/meshes/es200rn_120/visual/base_link.stl"/>
-            </geometry>
-            <material name="${prefix}visual_material">
-                <color rgba="${51.0/255.0} ${102.0/255.0} ${204.0/255.0} 1"/>
-            </material>
-        </visual>
-        <collision>
-            <geometry>
-                <mesh filename="package://motoman_es200rn_120_support/meshes/es200rn_120/collision/base_link.stl"/>
-            </geometry>
-            <material name="${prefix}collision_material">
-                <color rgba="${51.0/255.0} ${102.0/255.0} ${204.0/255.0} 1"/>
-            </material>
-        </collision>
+      <visual>
+        <origin xyz="0 0 0" rpy="0 0 0"/>
+        <geometry>
+          <mesh filename="package://motoman_es200rn_120_support/meshes/es200rn_120/visual/base_link.stl"/>
+        </geometry>
+        <material name="${prefix}visual_material">
+          <color rgba="${51.0/255.0} ${102.0/255.0} ${204.0/255.0} 1"/>
+        </material>
+      </visual>
+      <collision>
+        <geometry>
+          <mesh filename="package://motoman_es200rn_120_support/meshes/es200rn_120/collision/base_link.stl"/>
+        </geometry>
+        <material name="${prefix}collision_material">
+          <color rgba="${51.0/255.0} ${102.0/255.0} ${204.0/255.0} 1"/>
+        </material>
+      </collision>
     </link>
     <link name="${prefix}link_s">
-        <visual>
-            <origin xyz="0 0 0" rpy="0 0 0"/>
-            <geometry>
-                <mesh filename="package://motoman_es200rn_120_support/meshes/es200rn_120/visual/link_s.stl"/>
-            </geometry>
-            <material name="${prefix}visual_material"/>
-        </visual>
-        <collision>
-            <origin xyz="0 0 0" rpy="0 0 0"/>
-            <geometry>
-                <mesh filename="package://motoman_es200rn_120_support/meshes/es200rn_120/collision/link_s.stl"/>
-            </geometry>
-            <material name="${prefix}collision_material"/>
-        </collision>
+      <visual>
+        <origin xyz="0 0 0" rpy="0 0 0"/>
+        <geometry>
+          <mesh filename="package://motoman_es200rn_120_support/meshes/es200rn_120/visual/link_s.stl"/>
+        </geometry>
+        <material name="${prefix}visual_material"/>
+      </visual>
+      <collision>
+        <origin xyz="0 0 0" rpy="0 0 0"/>
+        <geometry>
+          <mesh filename="package://motoman_es200rn_120_support/meshes/es200rn_120/collision/link_s.stl"/>
+        </geometry>
+        <material name="${prefix}collision_material"/>
+      </collision>
     </link>
     <link name="${prefix}link_l">
-        <visual>
-            <origin xyz="0 0 0" rpy="0 0 0"/>
-            <geometry>
-                <mesh filename="package://motoman_es200rn_120_support/meshes/es200rn_120/visual/link_l.stl"/>
-            </geometry>
-            <material name="${prefix}visual_material"/>
-        </visual>
-        <collision>
-            <origin xyz="0 0 0" rpy="0 0 0"/>
-            <geometry>
-                <mesh filename="package://motoman_es200rn_120_support/meshes/es200rn_120/collision/link_l.stl"/>
-            </geometry>
-            <material name="${prefix}collision_material"/>
-        </collision>
+      <visual>
+        <origin xyz="0 0 0" rpy="0 0 0"/>
+        <geometry>
+          <mesh filename="package://motoman_es200rn_120_support/meshes/es200rn_120/visual/link_l.stl"/>
+        </geometry>
+        <material name="${prefix}visual_material"/>
+      </visual>
+      <collision>
+        <origin xyz="0 0 0" rpy="0 0 0"/>
+        <geometry>
+          <mesh filename="package://motoman_es200rn_120_support/meshes/es200rn_120/collision/link_l.stl"/>
+        </geometry>
+        <material name="${prefix}collision_material"/>
+      </collision>
     </link>
     <link name="${prefix}link_u">
-        <visual>
-            <origin xyz="0 0 0" rpy="0 0 0"/>
-            <geometry>
-                <mesh filename="package://motoman_es200rn_120_support/meshes/es200rn_120/visual/link_u.stl"/>
-            </geometry>
-            <material name="${prefix}visual_material"/>
-        </visual>
-        <collision>
-            <origin xyz="0 0 0" rpy="0 0 0"/>
-            <geometry>
-                <mesh filename="package://motoman_es200rn_120_support/meshes/es200rn_120/collision/link_u.stl"/>
-            </geometry>
-            <material name="${prefix}collision_material"/>
-        </collision>
+      <visual>
+        <origin xyz="0 0 0" rpy="0 0 0"/>
+        <geometry>
+          <mesh filename="package://motoman_es200rn_120_support/meshes/es200rn_120/visual/link_u.stl"/>
+        </geometry>
+        <material name="${prefix}visual_material"/>
+      </visual>
+      <collision>
+        <origin xyz="0 0 0" rpy="0 0 0"/>
+        <geometry>
+          <mesh filename="package://motoman_es200rn_120_support/meshes/es200rn_120/collision/link_u.stl"/>
+        </geometry>
+        <material name="${prefix}collision_material"/>
+      </collision>
     </link>
     <link name="${prefix}link_r">
-        <visual>
-            <origin xyz="0 0 0" rpy="0 0 0"/>
-            <geometry>
-                <mesh filename="package://motoman_es200rn_120_support/meshes/es200rn_120/visual/link_r.stl"/>
-            </geometry>
-            <material name="${prefix}visual_material"/>
-        </visual>
-        <collision>
-            <origin xyz="0 0 0" rpy="0 0 0"/>
-            <geometry>
-                <mesh filename="package://motoman_es200rn_120_support/meshes/es200rn_120/collision/link_r.stl"/>
-            </geometry>
-            <material name="${prefix}collision_material"/>
-        </collision>
+      <visual>
+        <origin xyz="0 0 0" rpy="0 0 0"/>
+        <geometry>
+          <mesh filename="package://motoman_es200rn_120_support/meshes/es200rn_120/visual/link_r.stl"/>
+        </geometry>
+        <material name="${prefix}visual_material"/>
+      </visual>
+      <collision>
+        <origin xyz="0 0 0" rpy="0 0 0"/>
+        <geometry>
+          <mesh filename="package://motoman_es200rn_120_support/meshes/es200rn_120/collision/link_r.stl"/>
+        </geometry>
+        <material name="${prefix}collision_material"/>
+      </collision>
     </link>
     <link name="${prefix}link_b">
-        <visual>
-            <origin xyz="0 0 0" rpy="0 0 0"/>
-            <geometry>
-                <mesh filename="package://motoman_es200rn_120_support/meshes/es200rn_120/visual/link_b.stl"/>
-            </geometry>
-            <material name="${prefix}visual_material"/>
-        </visual>
-        <collision>
-            <origin xyz="0 0 0" rpy="0 0 0"/>
-            <geometry>
-                <mesh filename="package://motoman_es200rn_120_support/meshes/es200rn_120/collision/link_b.stl"/>
-            </geometry>
-            <material name="${prefix}collision_material"/>
-        </collision>
+      <visual>
+        <origin xyz="0 0 0" rpy="0 0 0"/>
+        <geometry>
+          <mesh filename="package://motoman_es200rn_120_support/meshes/es200rn_120/visual/link_b.stl"/>
+        </geometry>
+        <material name="${prefix}visual_material"/>
+      </visual>
+      <collision>
+        <origin xyz="0 0 0" rpy="0 0 0"/>
+        <geometry>
+          <mesh filename="package://motoman_es200rn_120_support/meshes/es200rn_120/collision/link_b.stl"/>
+        </geometry>
+        <material name="${prefix}collision_material"/>
+      </collision>
     </link>
     <link name="${prefix}link_t">
-        <visual>
-            <origin xyz="0 0 0" rpy="0 0 0"/>
-            <geometry>
-                <mesh filename="package://motoman_es200rn_120_support/meshes/es200rn_120/visual/link_t.stl"/>
-            </geometry>
-            <material name="${prefix}visual_material"/>
-        </visual>
-        <collision>
-            <origin xyz="0 0 0" rpy="0 0 0"/>
-            <geometry>
-                <mesh filename="package://motoman_es200rn_120_support/meshes/es200rn_120/collision/link_t.stl"/>
-            </geometry>
-            <material name="${prefix}collision_material"/>
-        </collision>
+      <visual>
+        <origin xyz="0 0 0" rpy="0 0 0"/>
+        <geometry>
+          <mesh filename="package://motoman_es200rn_120_support/meshes/es200rn_120/visual/link_t.stl"/>
+        </geometry>
+        <material name="${prefix}visual_material"/>
+      </visual>
+      <collision>
+        <origin xyz="0 0 0" rpy="0 0 0"/>
+        <geometry>
+          <mesh filename="package://motoman_es200rn_120_support/meshes/es200rn_120/collision/link_t.stl"/>
+        </geometry>
+        <material name="${prefix}collision_material"/>
+      </collision>
     </link>
     <link name="${prefix}tool0"/>
     <link name="${prefix}balancer_piston">
-        <visual>
-            <origin xyz="0 0 0" rpy="0 0 0"/>
-            <geometry>
-                <mesh filename="package://motoman_es200rn_120_support/meshes/es200rn_120/visual/balancer_piston.stl"/>
-            </geometry>
-            <material name="${prefix}visual_material"/>
-        </visual>
-        <collision>
-            <origin xyz="0 0 0" rpy="0 0 0"/>
-            <geometry>
-                <mesh filename="package://motoman_es200rn_120_support/meshes/es200rn_120/collision/balancer_piston.stl"/>
-            </geometry>
-            <material name="${prefix}collision_material"/>
-        </collision>
+      <visual>
+        <origin xyz="0 0 0" rpy="0 0 0"/>
+        <geometry>
+          <mesh filename="package://motoman_es200rn_120_support/meshes/es200rn_120/visual/balancer_piston.stl"/>
+        </geometry>
+        <material name="${prefix}visual_material"/>
+      </visual>
+      <collision>
+        <origin xyz="0 0 0" rpy="0 0 0"/>
+        <geometry>
+          <mesh filename="package://motoman_es200rn_120_support/meshes/es200rn_120/collision/balancer_piston.stl"/>
+        </geometry>
+        <material name="${prefix}collision_material"/>
+      </collision>
     </link>
     <link name="${prefix}balancer_rod">
-        <visual>
-            <origin xyz="0 0 0" rpy="0 0 0"/>
-            <geometry>
-                <mesh filename="package://motoman_es200rn_120_support/meshes/es200rn_120/visual/balancer_rod.stl"/>
-            </geometry>
-            <material name="${prefix}visual_material"/>
-        </visual>
-        <collision>
-            <origin xyz="0 0 0" rpy="0 0 0"/>
-            <geometry>
-                <mesh filename="package://motoman_es200rn_120_support/meshes/es200rn_120/collision/balancer_rod.stl"/>
-            </geometry>
-            <material name="${prefix}collision_material"/>
-        </collision>
+      <visual>
+        <origin xyz="0 0 0" rpy="0 0 0"/>
+        <geometry>
+          <mesh filename="package://motoman_es200rn_120_support/meshes/es200rn_120/visual/balancer_rod.stl"/>
+        </geometry>
+        <material name="${prefix}visual_material"/>
+      </visual>
+      <collision>
+        <origin xyz="0 0 0" rpy="0 0 0"/>
+        <geometry>
+          <mesh filename="package://motoman_es200rn_120_support/meshes/es200rn_120/collision/balancer_rod.stl"/>
+        </geometry>
+        <material name="${prefix}collision_material"/>
+      </collision>
     </link>
     <!-- end of link list -->
     <!-- joint list -->
     <joint name="${prefix}joint_1" type="revolute">
-        <origin xyz="0 0 0" rpy="0 0 0"/>
-        <parent link="${prefix}base_link"/>
-        <child link="${prefix}link_s"/>
-        <axis xyz="0 0 1"/>
-        <limit lower="${radians(-180)}" upper="${radians(180)}" effort="0" velocity="${radians(90)}"/>
+      <origin xyz="0 0 0" rpy="0 0 0"/>
+      <parent link="${prefix}base_link"/>
+      <child link="${prefix}link_s"/>
+      <axis xyz="0 0 1"/>
+      <limit lower="${radians(-180)}" upper="${radians(180)}" effort="0" velocity="${radians(90)}"/>
     </joint>
     <joint name="${prefix}joint_2" type="revolute">
-        <origin xyz="0.740 0 0.450" rpy="0 ${radians(-90)} 0"/>
-        <parent link="${prefix}link_s"/>
-        <child link="${prefix}link_l"/>
-        <axis xyz="0 1 0"/>
-        <limit lower="${radians(-40)}" upper="${radians(170)}" effort="0" velocity="${radians(85)}"/>
+      <origin xyz="0.740 0 0.450" rpy="0 ${radians(-90)} 0"/>
+      <parent link="${prefix}link_s"/>
+      <child link="${prefix}link_l"/>
+      <axis xyz="0 1 0"/>
+      <limit lower="${radians(-40)}" upper="${radians(170)}" effort="0" velocity="${radians(85)}"/>
     </joint>
     <joint name="${prefix}joint_3" type="revolute">
-        <origin xyz="1.150 0 0" rpy="0 0 0"/>
-        <parent link="${prefix}link_l"/>
-        <child link="${prefix}link_u"/>
-        <axis xyz="0 1 0"/>
-        <limit lower="${radians(-180)}" upper="${radians(79.4)}" effort="0" velocity="${radians(85)}"/>
+      <origin xyz="1.150 0 0" rpy="0 0 0"/>
+      <parent link="${prefix}link_l"/>
+      <child link="${prefix}link_u"/>
+      <axis xyz="0 1 0"/>
+      <limit lower="${radians(-180)}" upper="${radians(79.4)}" effort="0" velocity="${radians(85)}"/>
     </joint>
     <joint name="${prefix}joint_4" type="revolute">
-        <origin xyz="0.250 0 0" rpy="0 0 0"/>
-        <parent link="${prefix}link_u"/>
-        <child link="${prefix}link_r"/>
-        <axis xyz="0 0 -1"/>
-        <limit lower="${radians(-360)}" upper="${radians(360)}" effort="0" velocity="${radians(175)}"/>
+      <origin xyz="0.250 0 0" rpy="0 0 0"/>
+      <parent link="${prefix}link_u"/>
+      <child link="${prefix}link_r"/>
+      <axis xyz="0 0 -1"/>
+      <limit lower="${radians(-360)}" upper="${radians(360)}" effort="0" velocity="${radians(175)}"/>
     </joint>
     <joint name="${prefix}joint_5" type="revolute">
-        <origin xyz="0 0 -2.100" rpy="0 0 0"/>
-        <parent link="${prefix}link_r"/>
-        <child link="${prefix}link_b"/>
-        <axis xyz="0 1 0"/>
-        <limit lower="${radians(-130)}" upper="${radians(130)}" effort="0" velocity="${radians(145)}"/>
+      <origin xyz="0 0 -2.100" rpy="0 0 0"/>
+      <parent link="${prefix}link_r"/>
+      <child link="${prefix}link_b"/>
+      <axis xyz="0 1 0"/>
+      <limit lower="${radians(-130)}" upper="${radians(130)}" effort="0" velocity="${radians(145)}"/>
     </joint>
     <joint name="${prefix}joint_6" type="revolute">
-        <origin xyz="0 0 -0.225" rpy="0 0 0"/>
-        <parent link="${prefix}link_b"/>
-        <child link="${prefix}link_t"/>
-        <axis xyz="0 0 -1"/>
-        <limit lower="${radians(-360)}" upper="${radians(360)}" effort="0" velocity="${radians(240)}"/>
+      <origin xyz="0 0 -0.225" rpy="0 0 0"/>
+      <parent link="${prefix}link_b"/>
+      <child link="${prefix}link_t"/>
+      <axis xyz="0 0 -1"/>
+      <limit lower="${radians(-360)}" upper="${radians(360)}" effort="0" velocity="${radians(240)}"/>
     </joint>
     <joint name="${prefix}joint_6-tool0" type="fixed">
-        <origin xyz="0 0 0" rpy="0 ${radians(180)} 0"/>
-        <parent link="${prefix}link_t"/>
-        <child link="${prefix}tool0"/>
+      <origin xyz="0 0 0" rpy="0 ${radians(180)} 0"/>
+      <parent link="${prefix}link_t"/>
+      <child link="${prefix}tool0"/>
     </joint>
     <joint name="${prefix}joint_balancer_piston" type="fixed">
-        <origin xyz="-0.260 0 0.770" rpy="0 0 0"/>
-        <parent link="${prefix}link_s"/>
-        <child link="${prefix}balancer_piston"/>
+      <origin xyz="-0.260 0 0.770" rpy="0 0 0"/>
+      <parent link="${prefix}link_s"/>
+      <child link="${prefix}balancer_piston"/>
     </joint>
     <joint name="${prefix}joint_balancer_rod" type="fixed">
-        <origin xyz="${0.740 + 0.220 * cos(radians(55))} 0 ${0.450 + 0.220 * sin(radians(55))}" rpy="0 0 0"/>
-        <parent link="${prefix}link_s"/>
-        <child link="${prefix}balancer_rod"/>
+      <origin xyz="${0.740 + 0.220 * cos(radians(55))} 0 ${0.450 + 0.220 * sin(radians(55))}" rpy="0 0 0"/>
+      <parent link="${prefix}link_s"/>
+      <child link="${prefix}balancer_rod"/>
     </joint>
     <!-- end of joint list -->
     <!-- ROS base_link to Robot Manufacturer World Coordinates transform -->
-    <link name="${prefix}base" />
+    <link name="${prefix}base"/>
     <joint name="${prefix}base_link-base" type="fixed">
-        <origin xyz="0 0 0" rpy="0 0 0"/>
-        <parent link="${prefix}base_link"/>
-        <child link="${prefix}base"/>
-    </joint>
-</xacro:macro>
+      <origin xyz="0 0 0" rpy="0 0 0"/>
+      <parent link="${prefix}base_link"/>
+      <child link="${prefix}base"/>
+    </joint>
+  </xacro:macro>
 </robot>
